File: devboard/devboard.kicad_pcb (KiCad board)
At the start: 2 copper layers, 100 x 100 mm, 58 parts, among them J1 Conn_02x12_Odd_Even, J10 Conn_01x06, J11 Conn_01x06, J12 Conn_01x04, J13 Conn_01x04, J14 Conn_01x03, J15 Conn_01x05, J16 Conn_01x03, J17 Conn_01x08, J18 Conn_01x03, J19 Conn_01x08, J2 Conn_02x12_Odd_Even, J20 Conn_02x05_Odd_Even, J21 Conn_01x08, J22 Conn_01x02, J23 Conn_01x10, J24 Barrel_Jack, J25 Conn_01x03, J26 Conn_01x03, J27 Conn_01x02, J28 Conn_01x02, J29 Conn_01x03, J3 Conn_02x12_Odd_Even, J30 Conn_01x04, J31 Conn_01x06, J32 Conn_01x08, J33 Conn_01x05, J34 Conn_01x03, J35 Conn_01x05, J36 Conn_01x05, J37 Conn_01x03, J38 Conn_01x08, J39 Conn_01x08, J4 Conn_02x12_Odd_Even, J40 Conn_01x10, J41 Conn_01x04, J42 Conn_01x03, J43 Conn_01x03, J5 Conn_01x05, J6 Conn_01x05, J7 Conn_01x05, J8 Conn_01x03, J9 Conn_01x06, U1 SN65HVD230, U2 SN65HVD230

Commit message: update devboard
Parts:
- added G***: LOGO, libs:distrap_logo_mini_9x9mm, F.Cu at (183.8, 59.5)
- added G***: LOGO, libs:distrap_qr_17x17, F.Cu at (142.2, 93.5)

Commit message: update stmstamp & devboard
Parts:
- removed J29, J34: Conn_01x03, Pin_Headers:Pin_Header_Straight_1x03_Pitch2.54mm
- J25, J26: value Conn_01x03 -> Conn_02x03_Odd_Even; footprint Pin_Headers:Pin_Header_Straight_1x03_Pitch2.54mm -> libs:CAN_Header
- moved J26 2.54 mm to (168.3, 132.8)
- moved G*** 0.71 mm to (142.7, 94.0)
- moved G*** 0.59 mm to (184.0, 60.0)
Connections:
- J25 pad 2: /CAN3_H -> /CAN3_L
- J25 pad 3: GND -> /CAN3_H
- J26 pad 2: /CAN1_H -> /CAN1_L
- J26 pad 3: GND -> /CAN1_H
- JP1 pad 1: /CAN3_L -> /CAN3_H
- JP2 pad 1: /CAN1_L -> /CAN1_H
- R5 pad 2: /CAN3_H -> /CAN3_L
- R6 pad 2: /CAN1_H -> /CAN1_L
- U1 pad 6: /CAN3_H -> /CAN3_L
- U1 pad 7: /CAN3_L -> /CAN3_H
- U2 pad 6: /CAN1_H -> /CAN1_L
- U2 pad 7: /CAN1_L -> /CAN1_H
Routing:
- net /CAN3_H: track 45.9 -> 40.8 mm
- net /CAN1_L: track 40.7 -> 43.9 mm
- net /CAN1_H: track 44.7 -> 47.3 mm
- net /GPIO1: track 84.3 -> 82.5 mm
- net /CAN3_L: track 48.7 -> 49.4 mm, vias 0 -> 1
- net GND: track 569.8 -> 570.5 mm
Other:
- outline, holes or cut-outs redrawn
