File: devboard/devboard.sch (KiCad schematic (older format))
At the start: 57 parts, among them J1 Conn_02x12_Odd_Even, J10 Conn_01x06, J11 Conn_01x06, J12 Conn_01x04, J13 Conn_01x04, J14 Conn_01x03, J15 Conn_01x05, J16 Conn_01x03, J17 Conn_01x08, J18 Conn_01x03, J19 Conn_01x08, J2 Conn_02x12_Odd_Even, J20 Conn_02x05_Odd_Even, J21 Conn_01x08, J22 Conn_01x02, J23 Conn_01x10, J24 Barrel_Jack, J25 Conn_01x03, J26 Conn_01x03, J27 Conn_01x02, J28 Conn_01x02, J29 Conn_01x03, J3 Conn_02x12_Odd_Even, J30 Conn_01x04, J31 Conn_01x06, J32 Conn_01x08, J33 Conn_01x05, J34 Conn_01x03, J35 Conn_01x05, J36 Conn_01x05, J37 Conn_01x03, J38 Conn_01x08, J39 Conn_01x08, J4 Conn_02x12_Odd_Even, J40 Conn_01x10, J41 Conn_01x04, J42 Conn_01x03, J43 Conn_01x03, J5 Conn_01x05, J6 Conn_01x05, J7 Conn_01x05, J8 Conn_01x03, J9 Conn_01x06, U1 SN65HVD230, U2 SN65HVD230

Commit message: update stmstamp & devboard
Parts:
- removed J25, J26, J29, J34: Conn_01x03, Pin_Headers:Pin_Header_Straight_1x03_Pitch2.54mm, symbol Conn_01x03
- added J25, J26: Conn_02x03_Odd_Even, Pin_Headers:Pin_Header_Straight_2x03_Pitch2.54mm, symbol Conn_02x03_Odd_Even
Changed lines of the file:
@@
 Wire Wire Line
 	18050 7850 19000 7850
-Text Label 18650 7850 0    60   ~ 0
+Text Label 18650 6800 0    60   ~ 0
 CAN3_H
 Connection ~ 18300 6800
-Text Label 18650 6800 0    60   ~ 0
+Text Label 18650 7850 0    60   ~ 0
 CAN3_L
 $Comp
@@
 	18300 7750 18300 7850
 Connection ~ 18300 7850
-$Comp
-L Conn_01x03 J25
-U 1 1 5A4C7746
-P 19750 7300
-F 0 "J25" H 19750 7500 50  0000 C CNN
-F 1 "Conn_01x03" H 19750 7100 50  0000 C CNN
-F 2 "Pin_Headers:Pin_Header_Straight_1x03_Pitch2.54mm" H 19750 7300 50  0001 C CNN
-F 3 "" H 19750 7300 50  0001 C CNN
-	1    19750 7300
-	1    0    0    -1
-$EndComp
 Wire Wire Line
 	19550 7200 19050 7200
@@
 Wire Wire Line
 	18050 9250 19000 9250
-Text Label 18650 9250 0    60   ~ 0
+Text Label 18650 8200 0    60   ~ 0
 CAN1_H
 Connection ~ 18300 8200
-Text Label 18650 8200 0    60   ~ 0
+Text Label 18650 9250 0    60   ~ 0
 CAN1_L
 $Comp
@@
 	18300 9150 18300 9250
 Connection ~ 18300 9250
-$Comp
-L Conn_01x03 J26
-U 1 1 5A4C8855
-P 19750 8700
-F 0 "J26" H 19750 8900 50  0000 C CNN
-F 1 "Conn_01x03" H 19750 8500 50  0000 C CNN
-F 2 "Pin_Headers:Pin_Header_Straight_1x03_Pitch2.54mm" H 19750 8700 50  0001 C CNN
-F 3 "" H 19750 8700 50  0001 C CNN
-	1    19750 8700
-	1    0    0    -1
-$EndComp
 Wire Wire Line
 	19550 8600 19050 8600
@@
 $EndComp
 $Comp
-L Conn_01x03 J29
-U 1 1 5A4E727A
-P 20800 7300
-F 0 "J29" H 20800 7500 50  0000 C CNN
-F 1 "Conn_01x03" H 20800 7100 50  0000 C CNN
-F 2 "Pin_Headers:Pin_Header_Straight_1x03_Pitch2.54mm" H 20800 7300 50  0001 C CNN
-F 3 "" H 20800 7300 50  0001 C CNN
-	1    20800 7300
-	1    0    0    -1
-$EndComp
-Wire Wire Line
-	20600 7200 20100 7200
-Wire Wire Line
-	20600 7300 20100 7300
-Wire Wire Line
-	20600 7400 20100 7400
-Wire Wire Line
-	20100 7400 20100 7550
-$Comp
 L GND #PWR050
 U 1 1 5A4E7284
-P 20100 7550
-F 0 "#PWR050" H 20100 7300 50  0001 C CNN
-F 1 "GND" H 20100 7400 50  0000 C CNN
-F 2 "" H 20100 7550 50  0001 C CNN
-F 3 "" H 20100 7550 50  0001 C CNN
-	1    20100 7550
+P 20600 7550
+F 0 "#PWR050" H 20600 7300 50  0001 C CNN
+F 1 "GND" H 20600 7400 50  0000 C CNN
+F 2 "" H 20600 7550 50  0001 C CNN
+F 3 "" H 20600 7550 50  0001 C CNN
+	1    20600 7550
 	-1   0    0    -1
 $EndComp
-Text Label 20100 7200 0    60   ~ 0
+Text Label 20250 7200 0    60   ~ 0
 CAN3_L
-Text Label 20100 7300 0    60   ~ 0
+Text Label 20250 7300 0    60   ~ 0
 CAN3_H
-$Comp
-L Conn_01x03 J34
-U 1 1 5A4E73A7
-P 20800 8700
-F 0 "J34" H 20800 8900 50  0000 C CNN
-F 1 "Conn_01x03" H 20800 8500 50  0000 C CNN
-F 2 "Pin_Headers:Pin_Header_Straight_1x03_Pitch2.54mm" H 20800 8700 50  0001 C CNN
-F 3 "" H 20800 8700 50  0001 C CNN
-	1    20800 8700
-	1    0    0    -1
-$EndComp
-Wire Wire Line
-	20600 8600 20100 8600
-Wire Wire Line
-	20600 8700 20100 8700
-Wire Wire Line
-	20600 8800 20100 8800
-Wire Wire Line
-	20100 8800 20100 8950
-$Comp
-L GND #PWR051
-U 1 1 5A4E73B1
-P 20100 8950
-F 0 "#PWR051" H 20100 8700 50  0001 C CNN
-F 1 "GND" H 20100 8800 50  0000 C CNN
-F 2 "" H 20100 8950 50  0001 C CNN
-F 3 "" H 20100 8950 50  0001 C CNN
-	1    20100 8950
-	-1   0    0    -1
-$EndComp
-Text Label 20100 8600 0    60   ~ 0
-CAN1_L
-Text Label 20100 8700 0    60   ~ 0
-CAN1_H
 $Comp
 L Conn_01x04 J30
@@
 	11550 7600 11550 7700
 $Comp
-L GND #PWR052
+L GND #PWR051
 U 1 1 5A4E98AF
 P 11550 7700
-F 0 "#PWR052" H 11550 7450 50  0001 C CNN
+F 0 "#PWR051" H 11550 7450 50  0001 C CNN
 F 1 "GND" H 11550 7550 50  0000 C CNN
 F 2 "" H 11550 7700 50  0001 C CNN
@@
 UART5_RX
 $Comp
-L GND #PWR053
+L GND #PWR052
 U 1 1 5A4F3B79
 P 9150 10200
-F 0 "#PWR053" H 9150 9950 50  0001 C CNN
+F 0 "#PWR052" H 9150 9950 50  0001 C CNN
 F 1 "GND" H 9150 10050 50  0000 C CNN
 F 2 "" H 9150 10200 50  0001 C CNN
@@
 	11550 8350 11550 8450
 $Comp
-L GND #PWR054
+L GND #PWR053
 U 1 1 5A4F4697
 P 11550 8450
-F 0 "#PWR054" H 11550 8200 50  0001 C CNN
+F 0 "#PWR053" H 11550 8200 50  0001 C CNN
 F 1 "GND" H 11550 8300 50  0000 C CNN
 F 2 "" H 11550 8450 50  0001 C CNN
@@
 	2800 11100 2800 11150
 $Comp
-L GND #PWR055
+L GND #PWR054
 U 1 1 5A4F52AD
 P 2800 11150
-F 0 "#PWR055" H 2800 10900 50  0001 C CNN
+F 0 "#PWR054" H 2800 10900 50  0001 C CNN
 F 1 "GND" H 2800 11000 50  0000 C CNN
 F 2 "" H 2800 11150 50  0001 C CNN
@@
 $EndComp
 $Comp
-L GND #PWR056
+L GND #PWR055
 U 1 1 5A4F7655
 P 15650 11400
-F 0 "#PWR056" H 15650 11150 50  0001 C CNN
+F 0 "#PWR055" H 15650 11150 50  0001 C CNN
 F 1 "GND" H 15650 11250 50  0000 C CNN
 F 2 "" H 15650 11400 50  0001 C CNN
@@
 Text Notes 650  4950 0    394  ~ 79
 DEVBOARD
+$Comp
+L Conn_02x03_Odd_Even J25
+U 1 1 5A5FB524
+P 19750 7300
+F 0 "J25" H 19800 7500 50  0000 C CNN
+F 1 "Conn_02x03_Odd_Even" H 19800 7100 50  0000 C CNN
+F 2 "Pin_Headers:Pin_Header_Straight_2x03_Pitch2.54mm" H 19750 7300 50  0001 C CNN
+F 3 "" H 19750 7300 50  0001 C CNN
+	1    19750 7300
+	1    0    0    -1
+$EndComp
+Wire Wire Line
+	20050 7200 20600 7200
+Wire Wire Line
+	20050 7300 20600 7300
+Wire Wire Line
+	20050 7400 20600 7400
+Wire Wire Line
+	20600 7400 20600 7550
+$Comp
+L Conn_02x03_Odd_Even J26
+U 1 1 5A5FC508
+P 19750 8700
+F 0 "J26" H 19800 8900 50  0000 C CNN
+F 1 "Conn_02x03_Odd_Even" H 19800 8500 50  0000 C CNN
+F 2 "Pin_Headers:Pin_Header_Straight_2x03_Pitch2.54mm" H 19750 8700 50  0001 C CNN
+F 3 "" H 19750 8700 50  0001 C CNN
+	1    19750 8700
+	1    0    0    -1
+$EndComp
+$Comp
+L GND #PWR056
+U 1 1 5A5FC8C2
+P 20600 8950
+F 0 "#PWR056" H 20600 8700 50  0001 C CNN
+F 1 "GND" H 20600 8800 50  0000 C CNN
+F 2 "" H 20600 8950 50  0001 C CNN
+F 3 "" H 20600 8950 50  0001 C CNN
+	1    20600 8950
+	-1   0    0    -1
+$EndComp
+Text Label 20250 8600 0    60   ~ 0
+CAN1_L
+Text Label 20250 8700 0    60   ~ 0
+CAN1_H
+Wire Wire Line
+	20050 8600 20600 8600
+Wire Wire Line
+	20050 8700 20600 8700
+Wire Wire Line
+	20050 8800 20600 8800
+Wire Wire Line
+	20600 8800 20600 8950
 $EndSCHEMATC
