File: stmstamp/stmstamp.kicad_pcb (KiCad board)
At the start: 2 copper layers, 50 x 50 mm, 39 parts, among them J1 Conn_02x12_Odd_Even, J2 Conn_02x12_Odd_Even, J3 Conn_02x12_Odd_Even, J4 Conn_02x12_Odd_Even, J5 Conn_02x05_Odd_Even, SW1 SW_Push, U1 STM32F756VGTx, U2 AP1117-33, Y1 Crystal_GND24

Commit message: stamp: logo & drc fixes
Parts:
- added REF***: OSHW-Logo2_14.6x12mm_SilkScreen, Symbols:OSHW-Logo2_14.6x12mm_SilkScreen, B.Cu at (145.0, 98.2)
Routing:
- net /GPIO2: track 14.5 -> 18.3 mm
- net GND: track 76.8 -> 78.9 mm
- net /NRST: track 60.2 -> 62.2 mm
- net +3V3: track 172.3 -> 174.2 mm
- net /SPI1_SCK: track 15.1 -> 13.7 mm
- net /TIM1_CH3N: track 19.4 -> 18.1 mm
- net /SPI3_SCK: track 26.9 -> 25.8 mm
- net /SPI2_MISO: track 16.9 -> 17.9 mm
- net /TIM3_CH4: track 23.0 -> 23.8 mm
- net /TIM2_CH2: track 16.9 -> 16.1 mm
- net /GPIO15: track 24.2 -> 24.9 mm
- net /TIM3_CH3: track 25.1 -> 25.7 mm

Commit message: update stmpstamp
Parts:
- added G***: LOGO, libs:distrap_logo_micro_5x7mm, F.Cu at (130.8, 88.5)
- added G***: LOGO, libs:base48_22x6, B.Cu at (145.2, 110.5)
- added G***: LOGO, libs:distrap_logo_full_17x18, B.Cu at (153.2, 97.0)
- added G***: LOGO, libs:haskell_11x8, B.Cu at (136.2, 88.0)
- moved REF*** 9.30 mm to (135.8, 99.5)

Commit message: update stmstamp & devboard
Connections:
- U1 pad 70: /CAN1_TX -> /CAN1_RX
- U1 pad 71: /CAN1_RX -> /CAN1_TX
Routing:
- net /CAN1_RX: track 37.1 -> 23.6 mm, vias 4 -> 1
- net /CAN1_TX: track 23.7 -> 29.3 mm, vias 1 -> 2
- net /TIM8_CH2: track 14.1 -> 14.8 mm
Other:
- board text added: "v2"
- board text removed: "v1"
