File: stmstamp/stmstamp.sch (KiCad schematic (older format))
At the start: 39 parts, among them J1 Conn_02x12_Odd_Even, J2 Conn_02x12_Odd_Even, J3 Conn_02x12_Odd_Even, J4 Conn_02x12_Odd_Even, J5 Conn_02x05_Odd_Even, SW1 SW_Push, U1 STM32F756VGTx, U2 AP1117-33, Y1 Crystal_GND24

Commit message: update stmstamp & devboard
Changed lines of the file:
@@
 Sheet 1 1
 Title "STMSTAMP"
-Date "2017-12-24"
-Rev "1"
+Date "2018-03-06"
+Rev "2"
 Comp "base48.cz"
 Comment1 ""
@@
 Text Label 6750 11650 0    60   ~ 0
 SPI1_MOSI
+Text Label 18100 8750 0    60   ~ 0
+CAN1_TX
 Text Label 18100 8650 0    60   ~ 0
-CAN1_TX
-Text Label 18100 8750 0    60   ~ 0
 CAN1_RX
 Text Label 6750 11250 0    60   ~ 0
