File: diffencB/diffencB.kicad_sch (KiCad schematic)
At the start: 13 parts, among them J1 RJ45_Shielded, U1 SN65LVDT41

Commit message: diffencB: v1
Parts:
- renumbered CLK to CLK1, CS to CS1, GND to GND1, MISO to MISO1
Connections:
- net at U1.11 (5B): now also J1.5; no longer J1.6
- net at U1.12 (5A): now also J1.4; no longer J1.5
- net at U1.17 (2Z): now also J1.6; no longer J1.4
Changed lines of the file:
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@@
+    (stroke (width 0) (type default))
+  )
+  (wire (pts (xy 165.1 88.9) (xy 165.1 101.6))
     (stroke (width 0) (type default))
   )
@@
     (stroke (width 0) (type default))
   )
+  (wire (pts (xy 165.1 88.9) (xy 172.72 88.9))
+    (stroke (width 0) (type default))
+  )
   (wire (pts (xy 142.24 113.03) (xy 161.29 113.03))
     (stroke (width 0) (type default))
@@
     (stroke (width 0) (type default))
   )
-  (wire (pts (xy 158.75 88.9) (xy 172.72 88.9))
-    (stroke (width 0) (type default))
-  )
   (wire (pts (xy 160.02 69.85) (xy 170.18 69.85))
     (stroke (width 0) (type default))
@@
     (stroke (width 0) (type default))
   )
+  (wire (pts (xy 172.72 91.44) (xy 166.37 91.44))
+    (stroke (width 0) (type default))
+  )
   (wire (pts (xy 44.45 160.02) (xy 44.45 166.37))
     (stroke (width 0) (type default))
   )
-  (wire (pts (xy 165.1 91.44) (xy 165.1 101.6))
-    (stroke (width 0) (type default))
-  )
   (wire (pts (xy 182.88 76.2) (xy 182.88 71.12))
     (stroke (width 0) (type default))
@@
     (stroke (width 0) (type default))
   )
-  (wire (pts (xy 166.37 93.98) (xy 166.37 104.14))
+  (wire (pts (xy 166.37 91.44) (xy 166.37 104.14))
     (stroke (width 0) (type default))
   )
@@
     (stroke (width 0) (type default))
   )
+  (wire (pts (xy 162.56 88.9) (xy 158.75 88.9))
+    (stroke (width 0) (type default))
+  )
   (wire (pts (xy 133.35 69.85) (xy 135.89 69.85))
     (stroke (width 0) (type default))
@@
     (stroke (width 0) (type default))
   )
+  (wire (pts (xy 172.72 93.98) (xy 162.56 93.98))
+    (stroke (width 0) (type default))
+  )
   (wire (pts (xy 128.27 86.36) (xy 140.97 86.36))
     (stroke (width 0) (type default))
   )
-  (wire (pts (xy 172.72 91.44) (xy 165.1 91.44))
-    (stroke (width 0) (type default))
-  )
-  (wire (pts (xy 172.72 93.98) (xy 166.37 93.98))
-    (stroke (width 0) (type default))
-  )
   (wire (pts (xy 140.97 83.82) (xy 139.7 83.82))
     (stroke (width 0) (type default))
   )
   (wire (pts (xy 158.75 83.82) (xy 172.72 83.82))
+    (stroke (width 0) (type default))
+  )
+  (wire (pts (xy 162.56 93.98) (xy 162.56 88.9))
     (stroke (width 0) (type default))
   )
@@
   (symbol (lib_id "Connector:Conn_01x01_Pin") (at 123.19 81.28 0) (unit 1)
     (in_bom yes) (on_board yes) (dnp no)
-    (property "Reference" "CLK" (at 123.19 80.01 0)
+    (property "Reference" "CLK1" (at 123.19 80.01 0)
       (effects (font (size 1.27 1.27)))
     )
@@
       (project "diffencB"
         (path "/327e9dcc-6600-417e-860c-ab0322827c90"
-          (reference "CLK") (unit 1)
+          (reference "CLK1") (unit 1)
         )
       )
@@
   (symbol (lib_id "Connector:Conn_01x01_Pin") (at 123.19 86.36 0) (unit 1)
     (in_bom yes) (on_board yes) (dnp no)
-    (property "Reference" "CS" (at 123.19 85.09 0)
+    (property "Reference" "CS1" (at 123.19 85.09 0)
       (effects (font (size 1.27 1.27)))
     )
@@
       (project "diffencB"
         (path "/327e9dcc-6600-417e-860c-ab0322827c90"
-          (reference "CS") (unit 1)
+          (reference "CS1") (unit 1)
         )
       )
@@
   (symbol (lib_id "Connector:Conn_01x01_Pin") (at 123.19 101.6 0) (unit 1)
     (in_bom yes) (on_board yes) (dnp no)
-    (property "Reference" "MISO" (at 123.19 100.33 0)
+    (property "Reference" "MISO1" (at 123.19 100.33 0)
       (effects (font (size 1.27 1.27)))
     )
@@
       (project "diffencB"
         (path "/327e9dcc-6600-417e-860c-ab0322827c90"
-          (reference "MISO") (unit 1)
+          (reference "MISO1") (unit 1)
         )
       )
@@
   (symbol (lib_id "Connector:Conn_01x01_Pin") (at 123.19 113.03 0) (unit 1)
     (in_bom yes) (on_board yes) (dnp no)
-    (property "Reference" "GND" (at 123.19 111.76 0)
+    (property "Reference" "GND1" (at 123.19 111.76 0)
       (effects (font (size 1.27 1.27)))
     )
@@
       (project "diffencB"
         (path "/327e9dcc-6600-417e-860c-ab0322827c90"
-          (reference "GND") (unit 1)
-        )
-      )
+          (reference "GND1") (unit 1)
+        )
+      )

Commit message: diffencB: diff pairs
Connections:
- net +3V3: now also J1.3; no longer J1.7
- net GND: now also J1.6; no longer J1.8
- net LVD2_N: now reaches J1.5
- net LVD2_N: now also U1.17 (2Z); no longer U1.11 (5B)
- net LVD2_P: now reaches J1.4
- net LVD2_P: now also U1.18 (2Y); no longer U1.12 (5A)
- net LVD1_N: now reaches J1.2, U1.19 (1Z)
- net LVD1_P: now reaches J1.1, U1.20 (1Y)
- new net LVD5_N: J1.8, U1.11 (5B)
- new net LVD5_P: J1.7, U1.12 (5A)
Changed lines of the file:
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@@
   (junction (at 139.7 93.98) (diameter 0) (color 0 0 0 0)
   )
-  (junction (at 170.18 113.03) (diameter 0) (color 0 0 0 0)
+  (junction (at 171.45 113.03) (diameter 0) (color 0 0 0 0)
   )
   (junction (at 135.89 69.85) (diameter 0) (color 0 0 0 0)
@@
     (stroke (width 0) (type default))
   )
-  (wire (pts (xy 195.58 113.03) (xy 170.18 113.03))
-    (stroke (width 0) (type default))
-  )
   (wire (pts (xy 158.75 81.28) (xy 172.72 81.28))
     (stroke (width 0) (type default))
   )
-  (wire (pts (xy 165.1 88.9) (xy 165.1 101.6))
+  (wire (pts (xy 158.75 86.36) (xy 170.18 86.36))
+    (stroke (width 0) (type default))
+  )
+  (wire (pts (xy 170.18 88.9) (xy 172.72 88.9))
     (stroke (width 0) (type default))
   )
@@
   )
   (wire (pts (xy 135.89 113.03) (xy 139.7 113.03))
-    (stroke (width 0) (type default))
-  )
-  (wire (pts (xy 170.18 96.52) (xy 170.18 69.85))
-    (stroke (width 0) (type default))
-  )
-  (wire (pts (xy 165.1 88.9) (xy 172.72 88.9))
     (stroke (width 0) (type default))
   )
@@
     (stroke (width 0) (type default))
   )
-  (wire (pts (xy 160.02 69.85) (xy 170.18 69.85))
+  (wire (pts (xy 172.72 93.98) (xy 171.45 93.98))
+    (stroke (width 0) (type default))
+  )
+  (wire (pts (xy 168.91 91.44) (xy 172.72 91.44))
+    (stroke (width 0) (type default))
+  )
+  (wire (pts (xy 160.02 69.85) (xy 171.45 69.85))
     (stroke (width 0) (type default))
   )
@@
     (stroke (width 0) (type default))
   )
-  (wire (pts (xy 161.29 113.03) (xy 170.18 113.03))
+  (wire (pts (xy 170.18 86.36) (xy 170.18 88.9))
     (stroke (width 0) (type default))
   )
-  (wire (pts (xy 158.75 86.36) (xy 172.72 86.36))
+  (wire (pts (xy 161.29 113.03) (xy 171.45 113.03))
     (stroke (width 0) (type default))
   )
-  (wire (pts (xy 172.72 91.44) (xy 166.37 91.44))
+  (wire (pts (xy 172.72 99.06) (xy 172.72 104.14))
     (stroke (width 0) (type default))
   )
   (wire (pts (xy 44.45 160.02) (xy 44.45 166.37))
+    (stroke (width 0) (type default))
+  )
+  (wire (pts (xy 171.45 86.36) (xy 171.45 69.85))
+    (stroke (width 0) (type default))
+  )
+  (wire (pts (xy 170.18 101.6) (xy 170.18 96.52))
+    (stroke (width 0) (type default))
+  )
+  (wire (pts (xy 172.72 86.36) (xy 171.45 86.36))
     (stroke (width 0) (type default))
   )
@@
     (stroke (width 0) (type default))
   )
+  (wire (pts (xy 168.91 88.9) (xy 168.91 91.44))
+    (stroke (width 0) (type default))
+  )
   (wire (pts (xy 135.89 69.85) (xy 160.02 69.85))
+    (stroke (width 0) (type default))
+  )
+  (wire (pts (xy 170.18 96.52) (xy 172.72 96.52))
     (stroke (width 0) (type default))
   )
@@
     (stroke (width 0) (type default))
   )
-  (wire (pts (xy 166.37 91.44) (xy 166.37 104.14))
-    (stroke (width 0) (type default))
-  )
   (wire (pts (xy 138.43 99.06) (xy 138.43 107.95))
     (stroke (width 0) (type default))
   )
-  (wire (pts (xy 166.37 104.14) (xy 158.75 104.14))
+  (wire (pts (xy 158.75 104.14) (xy 172.72 104.14))
     (stroke (width 0) (type default))
   )
-  (wire (pts (xy 172.72 96.52) (xy 170.18 96.52))
+  (wire (pts (xy 158.75 88.9) (xy 168.91 88.9))
     (stroke (width 0) (type default))
   )
-  (wire (pts (xy 162.56 88.9) (xy 158.75 88.9))
+  (wire (pts (xy 171.45 113.03) (xy 195.58 113.03))
     (stroke (width 0) (type default))
   )
@@
   )
   (wire (pts (xy 138.43 107.95) (xy 142.24 107.95))
-    (stroke (width 0) (type default))
-  )
-  (wire (pts (xy 172.72 93.98) (xy 162.56 93.98))
     (stroke (width 0) (type default))
   )
@@
     (stroke (width 0) (type default))
   )
-  (wire (pts (xy 162.56 93.98) (xy 162.56 88.9))
-    (stroke (width 0) (type default))
-  )
-  (wire (pts (xy 170.18 99.06) (xy 170.18 113.03))
+  (wire (pts (xy 171.45 93.98) (xy 171.45 113.03))
     (stroke (width 0) (type default))
   )
@@
     (stroke (width 0) (type default))
   )
-  (wire (pts (xy 172.72 99.06) (xy 170.18 99.06))
-    (stroke (width 0) (type default))
-  )
   (wire (pts (xy 135.89 88.9) (xy 140.97 88.9))
     (stroke (width 0) (type default))
   )
-  (wire (pts (xy 165.1 101.6) (xy 158.75 101.6))
+  (wire (pts (xy 158.75 101.6) (xy 170.18 101.6))
     (stroke (width 0) (type default))
   )
@@
     (stroke (width 0) (type default))
   )
+  (label "LVD5_N" (at 162.56 104.14 0) (fields_autoplaced)
+    (effects (font (size 1.27 1.27)) (justify left bottom))
+  )
+  (label "LVD2_P" (at 162.56 86.36 0) (fields_autoplaced)
+    (effects (font (size 1.27 1.27)) (justify left bottom))
+  )
+  (label "LVD1_P" (at 162.56 81.28 0) (fields_autoplaced)
+    (effects (font (size 1.27 1.27)) (justify left bottom))
+  )
+  (label "LVD1_N" (at 162.56 83.82 0) (fields_autoplaced)
+    (effects (font (size 1.27 1.27)) (justify left bottom))
+  )
+  (label "LVD2_N" (at 162.56 88.9 0) (fields_autoplaced)
+    (effects (font (size 1.27 1.27)) (justify left bottom))
+  )
+  (label "LVD5_P" (at 162.56 101.6 0) (fields_autoplaced)
+    (effects (font (size 1.27 1.27)) (justify left bottom))
+  )
   (symbol (lib_id "sn65lvdtxy:SN65LVDT41") (at 149.86 91.44 0) (unit 1)
